File: Hardware/MyDaq Breadboard.brd (EAGLE design)
At the start: 83.8 x 86.4 mm, 12 parts, among them U1 BREADBOARDCLEAR

Commit message: Centered logos and changed revision to symbol
Parts:
- added U$3: REVISION, SparkFun-Aesthetics:REVISION
- moved LOGO2 5.68 mm to (15.2, 80.0)
- moved LOGO1 4.58 mm to (15.2, 6.35)
Other:
- board text added: "H. Hoops"
- board text added: "T. Klopfenstein"
- board text removed: "H. Hoops, Revision by: T. Klopfenstein"
